Commit message: feat(arm_ik): 六轴运动学与逆解库
从URDF读取关节限位，输出六个舵机应转到的角度。核心依赖numpy+scipy，
不碰串口——硬件读写仍由cds_arm负责，两者通过ServoMap衔接。

模块：
- model/  自写URDF解析器（stdlib xml.etree）、SO(3) log/exp、STL读取
- kinematics/  FK与解析几何雅可比，共享一次链遍历
- solvers/  dls（自适应阻尼最小二乘，带限位钳制）与least_squares（scipy），
            经register_solver注册，可扩展
- servo/  关节弧度与CDS55xx tick互转，含URDF限位与舵机安全窗口的交集校验
- workspace/  可达空间采样与条件数分析
- trajectory/  关节/笛卡尔插值与时间参数化
- collision/  基于URDF box碰撞体的OBB自碰撞检测
- viz/  viser浏览器可视化，replay可读实机舵机驱动数字孪生

不可达目标返回限位内最接近的可达位姿而非报错：这台臂关节空间仅为±π六轴臂的
0.01%，可达域是一层壳（离基座38.9…350.9 mm），近似解比失败更有用。
IKResult.status为枚举而非布尔，调用方据此区分位置达标与姿态达标。

URDF修正：
- collision box与inertial对齐visual的rpy/xyz。原先尺寸照网格量取但未随visual
  旋转，kd_base的box中心偏移25 mm、y/z尺寸互换，finger_pinky有36.6 mm未被包住。
  修正值由scripts/audit_urdf_geometry.py从STL实测反算得出。
- 关节2限位由URDF与舵机安全窗口拟合修正（upper 0.4095→1.1670 rad）。
  标定残差从62.97°降至0.001°，dls求解器同步从299/300变为300/300收敛。

验证：46个测试通过，FK与yourdfpy在100组随机构型上一致到1e-16，
arm_ik的ruff与mypy均无告警。

Co-Authored-By: Claude Fable 5 <noreply@anthropic.com>

File: description/arm.urdf (robot description, URDF)
Before this commit: robot kd_u3b_uhand_arm, 17 links, 16 joints
Links:
- link finger_index: geometry collision box size=0.02882 0.03767 0.100769; visual mesh filename=meshes/finger_index.stl scale=0.001 0.001 0.001
- link finger_middle: geometry collision box size=0.038607 0.03767 0.106107; visual mesh filename=meshes/finger_middle.stl scale=0.001 0.001 0.001
- link finger_pinky: geometry collision box size=0.023195 0.03767 0.121367; visual mesh filename=meshes/finger_pinky.stl scale=0.001 0.001 0.001
- link finger_ring: geometry collision box size=0.03559 0.03767 0.10719; visual mesh filename=meshes/finger_ring.stl scale=0.001 0.001 0.001
- link finger_thumb: geometry collision box size=0.066936 0.046934 0.053096; visual mesh filename=meshes/finger_thumb.stl scale=0.001 0.001 0.001
- link hand_palm: geometry collision box size=0.111149 0.05531 0.084407; visual mesh filename=meshes/hand_palm.stl scale=0.001 0.001 0.001
- link kd_2: geometry collision box size=0.065 0.05 0.03; visual mesh filename=meshes/KD.STL scale=0.001 0.001 0.001
- link kd_3: geometry collision box size=0.050052 0.06504 0.03; visual mesh filename=meshes/KD.STL scale=0.001 0.001 0.001
- link kd_4: geometry collision box size=0.050052 0.06504 0.03; visual mesh filename=meshes/KD.STL scale=0.001 0.001 0.001
- link kd_base: geometry collision box size=0.065 0.03004 0.050024; visual mesh filename=meshes/KD.STL scale=0.001 0.001 0.001
- link kd_pair_front: geometry collision box size=0.050052 0.06504 0.03; visual mesh filename=meshes/KD.STL scale=0.001 0.001 0.001
- link kd_pair_rear: geometry collision box size=0.065 0.05 0.03; visual mesh filename=meshes/KD.STL scale=0.001 0.001 0.001
- link u3b_base: geometry collision box size=0.030131 0.055024 0.055048; visual mesh filename=meshes/U3B.STL scale=0.001 0.001 0.001
- link u3b_lower: geometry collision box size=0.055088 0.03 0.055088; visual mesh filename=meshes/U3B.STL scale=0.001 0.001 0.001
- link u3b_middle: geometry collision box size=0.055 0.03 0.055; visual mesh filename=meshes/U3B.STL scale=0.001 0.001 0.001
- link u3b_upper: geometry collision box size=0.030044 0.055111 0.055088; visual mesh filename=meshes/U3B.STL scale=0.001 0.001 0.001
Joints:
- joint kd_2_to_u3b_base: axis 0 1 0 -> 0 -1 0; limit lower=-0.4606 upper=0.4095 effort=6.0 velocity=2.0 -> lower=-0.4709 upper=1.1670 effort=6.0 velocity=2.0
- joint kd_base_side_to_kd_2: origin xyz=-0.0075 0.0 0.05 rpy=0 0 1.57 -> xyz=-0.0075 0.0 0.05 rpy=0 0 -1.57
- joint u3b_base_to_kd_3: origin xyz=0 0 0.045 -> xyz=0 0 0.045 rpy=0 0 3.14
